Commit message: added kdl compatible urdf

File: urdf/jackal_hulk.urdf.xacro (robot description, xacro)
@@ -10,4 +10,15 @@
     <color rgba="1 1 1 1"/>
   </material>
+<xacro:macro name="gazebo_reference" params="name color  mu1 mu2 kp kd selfcollide">
+    <gazebo reference="${name}">
+      <material>Gazebo/${color}</material>
+      <dampingFactor value="0.9"/>
+      <mu1 value="${mu1}"/>
+      <mu2 value="${mu2}"/>
+      <kp value="${kp}"/>
+      <kd value="${kd}"/>
+      <selfCollide value="${selfcollide}"/>
+    </gazebo>
+</xacro:macro>
  <xacro:macro name="default_inertial" params="mass">
     <inertial>
@@ -24,4 +35,12 @@
    </inertial>
   </xacro:macro>
+   <xacro:macro name="cuboid_inertia" params ="m l w h">
+  <inertial>
+   <mass value="${m}"/>
+   <inertia ixx="${m*(w*w + h*h)/12}"  ixy="0.0" ixz="0.0"
+            iyy="${m*(l*l + h*h)/12}"  iyz= "0.0"
+            izz="${m*(l*l + w*w)/12}"/>
+   </inertial>
+  </xacro:macro>
   <xacro:macro name="cylinder_inertia" params ="m r h">
   <inertial>
@@ -35,5 +54,5 @@
     <visual>
       <geometry>
-        <mesh filename="package://jackal/meshes/base_link.dae"/>
+        <mesh filename="package://jackal/meshes/jackal/base_link.dae"/>
       </geometry>
       <origin  rpy="0 0 0" xyz="0 0 0" />
@@ -43,5 +62,5 @@
       <origin  rpy="0 0 0" xyz="0 0 0"  />
       <geometry>
-        <mesh filename="package://jackal/meshes/base_link.dae"/>
+        <mesh filename="package://jackal/meshes/jackal/base_link.dae"/>
       </geometry>
     </collision>
@@ -55,8 +74,8 @@
     <material>Gazebo/Grey</material>
 </gazebo>
-<link name="link_1">
-    <visual>
-      <geometry>
-        <mesh filename="package://jackal/meshes/link_1.dae"/>
+<link name="dummy_link">
+    <visual>
+      <geometry>
+        <mesh filename="package://jackal/meshes/jackal/base_link.dae"/>
       </geometry>
       <origin  rpy="0 0 0" xyz="0 0 0" />
@@ -66,5 +85,35 @@
       <origin  rpy="0 0 0" xyz="0 0 0"  />
       <geometry>
-       <mesh filename="package://jackal/meshes/link_1.dae"/>
+        <mesh filename="package://jackal/meshes/jackal/base_link.dae"/>
+      </geometry>
+    </collision>
+    <xacro:cuboid_inertia m="10" l="0.25" w="0.25" h="0.25" />
+</link>
+<gazebo reference="dummy_link">
+    <static>0</static>
+    <mu1>1</mu1>
+    <mu2>1</mu2>
+    <selfCollide>true</selfCollide>
+    <material>Gazebo/Yellow</material>
+</gazebo>
+<joint name="dummy_joint" type="fixed">
+      <axis xyz="0 0 0"/>
+      <parent link="base_link"/>
+      <child link="dummy_link"/>
+      <origin xyz="0 0 0"/>
+</joint>
+<!-- This part of urdf is for Jackal Robot -->
+<link name="link_1">
+    <visual>
+      <geometry>
+        <mesh filename="package://jackal/meshes/jackal/link_1.dae"/>
+      </geometry>
+      <origin  rpy="0 0 0" xyz="0 0 0" />
+      <material name="blue"/>
+     </visual>
+    <collision>
+      <origin  rpy="0 0 0" xyz="0 0 0"  />
+      <geometry>
+       <mesh filename="package://jackal/meshes/jackal/link_1.dae"/>
       </geometry>
     </collision>
@@ -87,5 +136,5 @@
     <visual>
       <geometry>
-        <mesh filename="package://jackal/meshes/link_2.dae"/>
+        <mesh filename="package://jackal/meshes/jackal/link_2.dae"/>
       </geometry>
       <origin  rpy="0 0 0" xyz="0 0 0" />
@@ -95,5 +144,5 @@
       <origin  rpy="0 0 0" xyz="0 0 0"  />
       <geometry>
-       <mesh filename="package://jackal/meshes/link_2.dae"/>
+       <mesh filename="package://jackal/meshes/jackal/link_2.dae"/>
       </geometry>
     </collision>
@@ -128,5 +177,5 @@
     <visual>
       <geometry>
-        <mesh filename="package://jackal/meshes/link_2.dae"/>
+        <mesh filename="package://jackal/meshes/jackal/link_2.dae"/>
       </geometry>
       <origin  rpy="0 0 0" xyz="0 0 0" />
@@ -136,5 +185,5 @@
       <origin  rpy="0 0 0" xyz="0 0 0"  />
       <geometry>
-       <mesh filename="package://jackal/meshes/link_2.dae"/>
+       <mesh filename="package://jackal/meshes/jackal/link_2.dae"/>
       </geometry>
     </collision>
@@ -169,5 +218,5 @@
     <visual>
       <geometry>
-        <mesh filename="package://jackal/meshes/link_2.dae"/>
+        <mesh filename="package://jackal/meshes/jackal/link_2.dae"/>
       </geometry>
       <origin  rpy="0 0 0" xyz="0 0 0" />
@@ -177,5 +226,5 @@
       <origin  rpy="0 0 0" xyz="0 0 0"  />
       <geometry>
-       <mesh filename="package://jackal/meshes/link_2.dae"/>
+       <mesh filename="package://jackal/meshes/jackal/link_2.dae"/>
       </geometry>
     </collision>
@@ -210,5 +259,5 @@
     <visual>
       <geometry>
-        <mesh filename="package://jackal/meshes/link_2.dae"/>
+        <mesh filename="package://jackal/meshes/jackal/link_2.dae"/>
       </geometry>
       <origin  rpy="0 0 0" xyz="0 0 0" />
@@ -218,5 +267,5 @@
       <origin  rpy="0 0 0" xyz="0 0 0"  />
       <geometry>
-       <mesh filename="package://jackal/meshes/link_2.dae"/>
+       <mesh filename="package://jackal/meshes/jackal/link_2.dae"/>
       </geometry>
     </collision>
@@ -248,4 +297,486 @@
     </joint>
   </transmission>
+<!-- This part of urdf is for HULK robot ARM -->
+<joint name="ground_joint" type="fixed">
+    <parent link="base_link"/>
+    <child link="J0"/>
+    <origin rpy="0 0 1.57" xyz="0.12 0 0"/>
+</joint>
+<link
+    name="J0">
+    <inertial>
+      <origin
+        xyz="-0.000706 0.02721 0.001937"
+        rpy="0 0 0" />
+      <mass
+        value="0.842" />
+      <inertia
+        ixx="0.00064"
+        ixy="0"
+        ixz="0"
+        iyy="0"
+        iyz="0"
+        izz="0.00063" />
+    </inertial>
+    <visual>
+      <origin
+        xyz="0 0 0"
+        rpy="0 0 0" />
+      <geometry>
+        <mesh
+          filename="package://jackal/meshes/hulk/J0.dae" />
+      </geometry>
+      <material
+        name="">
+        <color
+          rgba="0.2509 0.25098 0.2509 1" />
+      </material>
+    </visual>
+    <collision>
+      <origin
+        xyz="-0.0007060 0.02720 0.00190"
+        rpy="0 0 0" />
+      <geometry>
+        <mesh
+          filename="package://jackal/meshes/hulk/J0.dae" />
+      </geometry>
+    </collision>
+</link>
+<xacro:gazebo_reference name="J0" color="White"  mu1="1" mu2="1" kp="10000" kd="1" selfcollide="True"/>
+  <link
+    name="J1">
+    <inertial>
+      <origin
+        xyz="0.01277 0.1058 0"
+        rpy="0 0 0" />
+      <mass
+        value="0.4427" />
+      <inertia
+        ixx="0.00087"
+        ixy="0.00012"
+        ixz="0"
+        iyy="0"
+        iyz="0"
+        izz="0.0008" />
+    </inertial>
+    <visual>
+      <origin
+        xyz="0 0 0"
+        rpy="0 0 0" />
+      <geometry>
+        <mesh
+          filename="package://jackal/meshes/hulk/J1.dae" />
+      </geometry>
+      <material
+        name="">
+        <color
+          rgba="1 1 1 1" />
+      </material>
+    </visual>
+    <collision>
+      <origin
+        xyz="0.01277 0.1056 0"
+        rpy="0 0 0" />
+      <geometry>
+        <mesh
+          filename="package://jackal/meshes/hulk/J1.dae" />
+      </geometry>
+    </collision>
+  </link>
+<xacro:gazebo_reference name="J1" color="White"  mu1="1" mu2="1" kp="10000" kd="1" selfcollide="True"/>
+  <joint
+    name="joint_6"
+    type="revolute">
+    <origin
+      xyz="0 0 0.1407"
+      rpy="1.57 0 3.14" />
+    <parent
+      link="J0" />
+    <child
+      link="J1" />
+    <axis
+      xyz="0 -1 0" />
+    <limit
+      effort="0.1"
+      velocity="0.5"
+      lower="-1.57"
+      upper="4.71"/>
+  </joint>
+<transmission name="link_joint_6_trans">
+      <type>transmission_interface/SimpleTransmission</type>
+      <actuator name="link_joint_6_motor">
+      <hardwareInterface>PositionJointInterface</hardwareInterface>
+        <mechanicalReduction>1</mechanicalReduction>
+      </actuator>
+      <joint name="joint_6">
+      <hardwareInterface>hardware_interface/PositionJointInterface</hardwareInterface>
+      </joint>
+ </transmission>
+  <link
+    name="J2">
+    <inertial>
+      <origin
+        xyz="-0.07434 0.1066 0"
+        rpy="0 0 0" />
+      <mass
+        value="0.3642" />
+      <inertia
+        ixx="0.0014"
+        ixy="-0.0004"
+        ixz="0"
+        iyy="0.0008"
+        iyz="0"
+        izz="0.0022" />
+    </inertial>
+    <visual>
+      <origin
+        xyz="0 0 0"
+        rpy="0 0 0" />
+      <geometry>
+        <mesh
+          filename="package://jackal/meshes/hulk/J2.dae" />
+      </geometry>
+      <material
+        name="">
+        <color
+          rgba="1 1 1 1" />
+      </material>
+    </visual>
+    <collision>
+      <origin
+        xyz="-0.0743 0.1066 0"
+        rpy="0 0 0" />
+      <geometry>
+        <mesh
+          filename="package://jackal/meshes/hulk/J2.dae" />
+      </geometry>
+    </collision>
+  </link>
+<xacro:gazebo_reference name="J2" color="White"  mu1="1" mu2="1" kp="10000" kd="1" selfcollide="True"/>
+  <joint
+    name="joint_7"
+    type="revolute">
+    <origin
+      xyz="-0.085 0.065 0"
+      rpy="0 0 0" />
+    <parent
+      link="J1" />
+    <child
+      link="J2" />
+    <axis
+      xyz="-1 0 0" />
+    <limit
+      effort="0.1"
+      velocity="0.5"
+      lower="-0.2"
+      upper="1.57"/>
+  </joint>
+<transmission name="link_joint_7_trans">
+      <type>transmission_interface/SimpleTransmission</type>
+      <actuator name="link_joint_7_motor">
+      <hardwareInterface>PositionJointInterface</hardwareInterface>
+        <mechanicalReduction>1</mechanicalReduction>
+      </actuator>
+      <joint name="joint_7">
+      <hardwareInterface>hardware_interface/PositionJointInterface</hardwareInterface>
+      </joint>
+ </transmission>
+  <link
+    name="J3">
+    <inertial>
+      <origin
+        xyz="-0.0092 0.00658 -4.E-09"
+        rpy="0 0 0" />
+      <mass
+        value="0.3458" />
+      <inertia
+        ixx="0"
+        ixy="0"
+        ixz="0"
+        iyy="0.0002"
+        iyz="0"
+        izz="0.0002" />
+    </inertial>
+    <visual>
+      <origin
+        xyz="0 0 0"
+        rpy="0 0 0" />
+      <geometry>
+        <mesh
+          filename="package://jackal/meshes/hulk/J3.dae" />
+      </geometry>
+      <material
+        name="">
+        <color
+          rgba="1 1 1 1" />
+      </material>
+    </visual>
+    <collision>
+      <origin
+        xyz="-0.00926 0.0065 0"
+        rpy="0 0 0" />
+      <geometry>
+        <mesh
+          filename="package://jackal/meshes/hulk/J3.dae" />
+      </geometry>
+    </collision>
+  </link>
+<xacro:gazebo_reference name="J3" color="White"  mu1="1" mu2="1" kp="10000" kd="1" selfcollide="True"/>
+  <joint
+    name="joint_8"
+    type="revolute">
+    <origin
+      xyz="0.08502 0.25 0"
+      rpy="0 0 0" />
+    <parent
+      link="J2" />
+    <child
+      link="J3" />
+    <axis
+      xyz="-1 0 0" />
+    <limit
+      effort="0.1"
+      velocity="0.5"
+      lower="0"
+      upper="2.2"/>
+  </joint>
+<transmission name="link_joint_8_trans">
+      <type>transmission_interface/SimpleTransmission</type>
+      <actuator name="link_joint_8_motor">
+      <hardwareInterface>PositionJointInterface</hardwareInterface>
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
Commit message: changed joint limits for better IK results

File: urdf/jackal_hulk.urdf.xacro (robot description, xacro)
@@ -469,5 +469,5 @@
       effort="0.1"
       velocity="0.5"
-      lower="-0.2"
+      lower="-1.57"
       upper="1.57"/>
   </joint>
@@ -538,5 +538,5 @@
       effort="0.1"
       velocity="0.5"
-      lower="0"
+      lower="-1.57"
       upper="2.2"/>
   </joint>
@@ -677,5 +677,5 @@
       velocity="0.5"
       lower="-3.14"
-      upper="0.785"/>
+      upper="3.14"/>
   </joint>
 <transmission name="link_joint_10_trans">
@@ -745,6 +745,6 @@
       effort="0.1"
       velocity="0.5"
-      lower="0"
-      upper="6.28"/>
+      lower="-3.14"
+      upper="3.14"/>
   </joint>
 <transmission name="link_joint_11_trans">

File: urdf/robot.urdf (robot description, URDF)
Before this commit: robot Hulk1_0, 9 links, 8 joints
Joints:
- joint joint_1: limit lower=-0.2 upper=1.57 effort=0.1 velocity=0.5 -> lower=-1.57 upper=1.57 effort=0.1 velocity=0.5
- joint joint_2: limit lower=0 upper=2.2 effort=0.1 velocity=0.5 -> lower=-1.57 upper=2.2 effort=0.1 velocity=0.5
- joint joint_4: limit lower=-3.14 upper=0.785 effort=0.1 velocity=0.5 -> lower=-3.14 upper=3.14 effort=0.1 velocity=0.5
- joint joint_5: limit lower=0 upper=6.28 effort=0.1 velocity=0.5 -> lower=-3.14 upper=3.14 effort=0.1 velocity=0.5
