Commit message: added dummy link

File: urdf/robot.urdf (robot description, URDF)
Before this commit: robot Hulk1_0, 9 links, 8 joints
Links:
- added link dummy_link; collision box size=0.01 0.01 0.01; visual box size=0.01 0.01 0.01
Joints:
- added joint dummy_joint: type fixed, parent base_link, child dummy_link, origin xyz=0.12 0 -0.250 rpy=0 0 0
